Commit message: updated values for robot

File: docs/urdf/robotarm.urdf (robot description, URDF)
Before this commit: robot robotarm, 5 links, 4 joints
Joints:
- joint axis1: axis 0 0 -1 -> 0 0 1; limit lower=-6.2831853 upper=6.2831853 effort=1 velocity=1 -> lower=-2.80 upper=2.80 effort=8 velocity=25
- joint axis2: axis 0 0 -1 -> 0 0 1; limit lower=-6.2831853 upper=6.2831853 effort=1 velocity=1 -> lower=-2.80 upper=0.35 effort=30 velocity=25
- joint axis3: axis 0 0 -1 -> 0 0 1; limit lower=-6.2831853 upper=6.2831853 effort=1 velocity=1 -> lower=-2.01 upper=2.36 effort=12 velocity=25
